File: upperboard/pcb/profi506_avr_kbd.sch (EAGLE design)
At the start: 14 parts, among them IC1 ATMEGA328-QFP32, IC2 DIP40 socket, Q1 16MHz

Commit message: new pcb v1.1 for avr kbd controller, added CS signal, added leds to indicate power status and activity
Parts:
- added LED1: PWR, adafruit:LEDCHIPLED_0805
- added LED2: BUSY, adafruit:LEDCHIPLED_0805
- added R8: 100, rcl:R-EU_R0805
- added R9: 200, rcl:R-EU_R0805
- R3: value 100 -> 470
- R4: value 200 -> 470
Connections:
- net AVR_CLK renamed AVR_MOSI
- net AVR_DAT renamed AVR_SCK
- removed net AVR_RST: IC2.5, R3.2, R4.2
- new net AVR_BUSY: IC1.PD6(AIN0), R4.2
- new net AVR_SS: IC2.4, R8.2, R9.2
- new net N$3: IC1.PD7(AIN1), R8.1
- new net N$4: LED1.A, R3.1
- new net N$5: LED2.A, R4.1
- net GND: now also LED1.C, LED2.C, R9.1; no longer R4.1
- net MISO: now also IC2.5; no longer R3.1
- net VCC: now also R3.2
Other:
- moved on the sheet: R3, R4
